File: hardware/pcb/tussenstukpw22/tussenstukpw22.kicad_sch (KiCad schematic)
At the start: 2 parts, among them J1 Conn_01x10, J2 Conn_01x10

Commit message: pcb updated
Connections:
- removed net GND1: J1.3 (Pin_3), J1.4 (Pin_4), J2.3 (Pin_3), J2.4 (Pin_4)
- removed net GND2: J1.7 (Pin_7), J1.8 (Pin_8), J2.7 (Pin_7), J2.8 (Pin_8)
- net GPIO1: no longer names the net of J1.2 (Pin_2)
- net GPIO1: no longer J2.1 (Pin_1)
- net GPIO2: no longer names the net of J1.10 (Pin_10)
- net GPIO2: no longer J2.9 (Pin_9)
- net SDA: no longer names the net of J1.6 (Pin_6)
- net SDA: no longer J2.5 (Pin_5)
- net SDL: no longer names the net of J1.5 (Pin_5)
- net SDL: no longer J2.6 (Pin_6)
- net VCC1: no longer names the net of J1.1 (Pin_1)
- net VCC1: no longer J2.2 (Pin_2)
- net VCC2: no longer names the net of J1.9 (Pin_9)
- net VCC2: no longer J2.10 (Pin_10)
Other:
- title: (none) -> Verbindingsstuk leafs
- moved on the sheet: J1, J2

Commit message: modified pcb
Parts:
- J1, J2: footprint Connector_PinHeader_2.00mm:PinHeader_2x05_P2.00mm_Vertical -> Connector_PinHeader_2.54mm:PinHeader_2x05_P2.54mm_Vertical
Connections:
- net GND: now reaches J1.1 (Pin_1)
- net GND: now also J1.9 (Pin_9), J2.1 (Pin_1), J2.9 (Pin_9)
- net +24V: now reaches J1.10 (Pin_10)
- net +24V: now also J1.2 (Pin_2), J2.10 (Pin_10), J2.2 (Pin_2)
- net SDA: now reaches J1.3 (Pin_3)
- net SDA: now also J1.7 (Pin_7), J2.3 (Pin_3), J2.7 (Pin_7)
- net SCL: now reaches J1.4 (Pin_4)
- net SCL: now also J1.8 (Pin_8), J2.4 (Pin_4), J2.8 (Pin_8)
- net SEL: now reaches J1.5 (Pin_5)
- net SEL: now also J1.6 (Pin_6), J2.5 (Pin_5), J2.6 (Pin_6)
Other:
- note removed: "Op J2: 2 & 10 = VCC 4 & 8 = GND 5 & 6 = SDA & SCL 1 & 9 = GPIO 7 & 3 = NOT CONNECTED (DUS DOORVERBONDEN MET GROUND 1 & 9 3 & 7 2 & 10 4 & 8 5 APART 6 APART LR 12 21 34 43 56 65 78 87 9 10 10 9"
- moved on the sheet: J2
