File: hardware/pcb/tussenstukpw22/tussenstukpw22.kicad_pcb (KiCad board)
At the start: 2 copper layers, 23 x 12 mm, 3 parts, among them J1 Conn_01x10, J2 Conn_01x10

Commit message: modified pcb
Parts:
- removed kibuzzard-62161CB7: G***, kibuzzard-62161CB7
- J1, J2: footprint Connector_PinHeader_2.00mm:PinHeader_2x05_P2.00mm_Vertical -> Connector_PinHeader_2.54mm:PinHeader_2x05_P2.54mm_Vertical
- moved J1 26.2 mm to (166.2, 93.4)
- moved J2 19.3 mm to (181.2, 103.5), turned to 180 degrees
Connections:
- J1 pad 1: /VCC1 -> GND
- J1 pad 10: /GPIO2 -> +24V
- J1 pad 2: /GPIO1 -> +24V
- J1 pad 3: /GND1 -> /SDA
- J1 pad 4: /GND1 -> /SCL
- J1 pad 5: /SDL -> /SEL
- J1 pad 6: /SDA -> /SEL
- J1 pad 7: /GND2 -> /SDA
- J1 pad 8: /GND2 -> /SCL
- J1 pad 9: /VCC2 -> GND
- J2 pad 1: /GPIO1 -> GND
- J2 pad 10: /VCC2 -> +24V
- J2 pad 2: /VCC1 -> +24V
- J2 pad 3: /GND1 -> /SDA
- J2 pad 4: /GND1 -> /SCL
- J2 pad 5: /SDA -> /SEL
- J2 pad 6: /SDL -> /SEL
- J2 pad 7: /GND2 -> /SDA
- J2 pad 8: /GND2 -> /SCL
- J2 pad 9: /GPIO2 -> GND
Routing:
- net /GND2: track 40.8 -> 0.00 mm
- net /GND1: track 40.8 -> 0.00 mm
- net /SDL: track 19.8 -> 0.00 mm
- net /VCC2: track 19.8 -> 0.00 mm
- net /VCC1: track 19.8 -> 0.00 mm
- net /SCL: track 0.00 -> 19.7 mm
- net +24V: track 0.00 -> 19.7 mm
- net /SDA: track 15.0 -> 31.8 mm
- net /GPIO2: track 15.0 -> 0.00 mm
- net /GPIO1: track 15.0 -> 0.00 mm
- net /SEL: track 0.00 -> 14.9 mm
- added copper zone on F.Cu, net GND
Other:
- board size 23 x 12 mm -> 21.5 x 17 mm
- board text removed: "Op J2: 2 & 10 = VCC 4 & 8 = GND 5 & 6 = SDA & SCL 1 & 9 = GPIO 7 & 3 = NOT CONNECTED (DUS DOORVERBONDEN MET GROUND 1 & 9 3 & 7 2 & 10 4 & 8 5 APART 6 APART LR 12 21 34 43 56 65 78 87 9 10 10 9"

Commit message: updated pcb
Changed lines of the file:
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@@
       (outputformat 1)
       (mirror false)
-      (drillshape 1)
+      (drillshape 0)
       (scaleselection 1)
-      (outputdirectory "")
+      (outputdirectory "../../../../../../../Users/jensv/Desktop/bestelling/tussenstuk/")
     )
   )
@@
   (segment (start 168.785 100.995) (end 178.645 100.995) (width 0.25) (layer "F.Cu") (net 4))
   (segment (start 178.645 100.995) (end 178.65 100.99) (width 0.25) (layer "F.Cu") (net 4))
+  (segment (start 178.645 98.455) (end 178.65 98.45) (width 0.25) (layer "F.Cu") (net 5))
+  (segment (start 166.245 98.455) (end 168.785 98.455) (width 0.25) (layer "F.Cu") (net 5))
+  (segment (start 178.65 98.45) (end 181.19 98.45) (width 0.25) (layer "F.Cu") (net 5))
   (segment (start 168.785 98.455) (end 178.645 98.455) (width 0.25) (layer "F.Cu") (net 5))
-  (segment (start 166.245 98.455) (end 168.785 98.455) (width 0.25) (layer "F.Cu") (net 5))
-  (segment (start 178.645 98.455) (end 178.65 98.45) (width 0.25) (layer "F.Cu") (net 5))
-  (segment (start 178.65 98.45) (end 181.19 98.45) (width 0.25) (layer "F.Cu") (net 5))
   (zone (net 1) (net_name "GND") (layer "F.Cu") (hatch edge 0.508)
     (connect_pads (clearance 0.508))
@@
       (pts
         (xy 184.5 107)
-        (xy 163.25 107)
-        (xy 163.25 90)
+        (xy 163 107)
+        (xy 163 90)
         (xy 184.5 90)
       )

Commit message: changes pcb
Routing:
- added copper zone on B.Cu, net GND
Changed lines of the file:
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@@
       (drillshape 0)
       (scaleselection 1)
-      (outputdirectory "../../../../../../../Users/jensv/Desktop/bestelling/tussenstuk/")
+      (outputdirectory "../../../../../../../Users/jensv/Desktop/tussenstuk/")
     )
   )
@@
   )
   (gr_rect (start 163 90) (end 184.5 107) (layer "Edge.Cuts") (width 0.1) (fill none))
-  (segment (start 168.785 93.375) (end 178.645 93.375) (width 2) (layer "F.Cu") (net 2))
-  (segment (start 178.645 103.535) (end 178.65 103.53) (width 2) (layer "F.Cu") (net 2))
-  (segment (start 168.785 103.535) (end 178.645 103.535) (width 2) (layer "F.Cu") (net 2))
-  (segment (start 178.645 93.375) (end 178.65 93.37) (width 2) (layer "F.Cu") (net 2))
+  (segment (start 168.785 103.535) (end 178.645 103.535) (width 2) (layer "B.Cu") (net 2))
+  (segment (start 178.645 103.535) (end 178.65 103.53) (width 2) (layer "B.Cu") (net 2))
+  (segment (start 168.785 93.375) (end 178.645 93.375) (width 2) (layer "B.Cu") (net 2))
+  (segment (start 178.645 93.375) (end 178.65 93.37) (width 2) (layer "B.Cu") (net 2))
   (segment (start 180.015489 99.815489) (end 181.19 100.99) (width 0.25) (layer "F.Cu") (net 3))
   (segment (start 167.424511 99.815489) (end 180.015489 99.815489) (width 0.25) (layer "F.Cu") (net 3))
@@
   (segment (start 168.785 98.455) (end 178.645 98.455) (width 0.25) (layer "F.Cu") (net 5))
   (zone (net 1) (net_name "GND") (layer "F.Cu") (hatch edge 0.508)
-    (connect_pads (clearance 0.508))
-    (min_thickness 0.254) (filled_areas_thickness no)
+    (connect_pads (clearance 0.2))
+    (min_thickness 0.1) (filled_areas_thickness no)
     (fill yes (thermal_gap 0.508) (thermal_bridge_width 1.5))
     (polygon
@@
         (xy 163 90)
         (xy 184.5 90)
+      )
+    )
+  )
+  (zone (net 1) (net_name "GND") (layer "B.Cu") (hatch edge 0.508)
+    (connect_pads (clearance 0.2))
+    (min_thickness 0.1) (filled_areas_thickness no)
+    (fill yes (thermal_gap 0.508) (thermal_bridge_width 1.5))
+    (polygon
+      (pts
+        (xy 184.5 107)
+        (xy 163 107.01)
+        (xy 163 90)
+        (xy 184.5 90)
