File: hardware/pcb/pcb_v1/pcb_v1.kicad_pcb (KiCad board)
At the start: 2 copper layers, 181.4 x 151.5 mm, 44 parts, among them J1 Conn_01x10, J2 Conn_01x10, J3 Conn_01x10, J4 Conn_01x10, J5 Conn_01x10, J6 Conn_01x10, U1 Pico, U2 TL2575-05

Commit message: worked on pcbv1
Parts:
- added J7: Barrel_Jack_Switch, Connector_BarrelJack:BarrelJack_CLIFF_FC681465S_SMT_Horizontal, B.Cu at (72.8, 171.9)
- added J8: Conn_01x05, Connector_PinSocket_2.54mm:PinSocket_1x05_P2.54mm_Horizontal, B.Cu at (138.8, 128.2)
- added R1: 3.1k, Resistor_SMD:R_0805_2012Metric, B.Cu at (194.5, 52.9)
- added R2: 1k, Resistor_SMD:R_0805_2012Metric, B.Cu at (198.2, 52.9)
- added REF**: Logo_Lannooleaf, Logo:Logo_Lannooleaf, B.Cu at (114.0, 148.0)
- added kibuzzard-6233C5FE: G***, kibuzzard-6233C5FE, B.Cu at (135.5, 156.5)
- added kibuzzard-6233C627: G***, kibuzzard-6233C627, B.Cu at (121.0, 156.5)
- added kibuzzard-6233C655: G***, kibuzzard-6233C655, B.Cu at (106.5, 156.6)
- added kibuzzard-6233C670: G***, kibuzzard-6233C670, B.Cu at (92.8, 156.6)
- added kibuzzard-6233C79C: G***, kibuzzard-6233C79C, B.Cu at (128.4, 81.6)
- added kibuzzard-6233C7BC: G***, kibuzzard-6233C7BC, B.Cu at (135.8, 81.1)
- C18: value 330uF -> 220uF
- D17: value 1N5819 -> 1N5822; footprint Diode_THT:D_DO-41_SOD81_P10.16mm_Horizontal -> Diode_THT:D_DO-201AD_P15.24mm_Horizontal
- L1: value 330uH -> 33uH
- U2: value TL2575-05 -> LM2596S-ADJ
- moved C18 86.1 mm to (189.7, 45.1), turned to 0 degrees
- moved L1 59.7 mm to (185.7, 57.8), turned to 90 degrees
- moved U2 48.9 mm to (201.2, 61.1), turned to 0 degrees
- moved D17 28.2 mm to (175.5, 68.1)
- moved C17 27.6 mm to (192.2, 71.4), turned to 180 degrees
- moved C12 8.78 mm to (200.7, 37.8), turned to 0 degrees
- moved U1 6.02 mm to (156.3, 103.8)
- moved C7 4.74 mm to (168.8, 135.7), turned to -90 degrees
- moved C1 4.61 mm to (130.7, 115.4), turned to 90 degrees
- moved C13 1.67 mm to (167.8, 38.3)
- moved C11 1.67 mm to (223.3, 49.3)
- moved C8 1.66 mm to (179.2, 115.9)
- moved C5 1.65 mm to (122.0, 166.0)
- moved C9 1.63 mm to (180.0, 84.0)
- moved C6 1.62 mm to (140.6, 161.0)
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Connections:
- J1 pad 1: /SDA -> GND
- J1 pad 10: /SCL -> +24V
- J1 pad 2: /SCL -> +24V
- J1 pad 3: +24V -> /SDA
- J1 pad 4: GND -> /SCL
- J1 pad 7: +24V -> /SDA
- J1 pad 8: GND -> /SCL
- J1 pad 9: /SDA -> GND
- J2 pad 1: /SDA -> GND
- J2 pad 10: /SCL -> +24V
- J2 pad 2: /SCL -> +24V
- J2 pad 3: +24V -> /SDA
- J2 pad 4: GND -> /SCL
- J2 pad 7: +24V -> /SDA
- J2 pad 8: GND -> /SCL
- J2 pad 9: /SDA -> GND
- J3 pad 1: /SDA -> GND
- J3 pad 10: /SCL -> +24V
- J3 pad 2: /SCL -> +24V
- J3 pad 3: +24V -> /SDA
- J3 pad 4: GND -> /SCL
- J3 pad 7: +24V -> /SDA
- J3 pad 8: GND -> /SCL
- J3 pad 9: /SDA -> GND
- J4 pad 1: /SDA -> GND
- J4 pad 10: /SCL -> +24V
- J4 pad 2: /SCL -> +24V
- J4 pad 3: +24V -> /SDA
- J4 pad 4: GND -> /SCL
- J4 pad 7: +24V -> /SDA
- J4 pad 8: GND -> /SCL
- J4 pad 9: /SDA -> GND
- J5 pad 1: /SDA -> GND
- J5 pad 10: /SCL -> +24V
- J5 pad 2: /SCL -> +24V
- J5 pad 3: +24V -> /SDA
- J5 pad 4: GND -> /SCL
- J5 pad 7: +24V -> /SDA
- J5 pad 8: GND -> /SCL
- J5 pad 9: /SDA -> GND
- J6 pad 1: /SDA -> GND
- J6 pad 10: /SCL -> +24V
- J6 pad 2: /SCL -> +24V
- J6 pad 3: +24V -> /SDA
- J6 pad 4: GND -> /SCL
- J6 pad 7: +24V -> /SDA
- J6 pad 8: GND -> /SCL
- J6 pad 9: /SDA -> GND
- U1 pad 1: /SEL3 -> /RX
- U1 pad 11: unconnected-(U1-Pad11) -> /SDA
- U1 pad 12: unconnected-(U1-Pad12) -> /SCL
- U1 pad 2: /SEL2 -> /CS
- U1 pad 22: /SEL4 -> unconnected-(U1-Pad22)
- U1 pad 24: unconnected-(U1-Pad24) -> /SEL4
- U1 pad 31: /SDA -> unconnected-(U1-Pad31)
- U1 pad 32: /SCL -> unconnected-(U1-Pad32)
- U1 pad 34: unconnected-(U1-Pad34) -> /SEL3
- U1 pad 4: /SEL1 -> /CSK
- U1 pad 5: unconnected-(U1-Pad5) -> /TX
- U1 pad 7: unconnected-(U1-Pad7) -> /SEL2
- U1 pad 9: unconnected-(U1-Pad9) -> /SEL1
- U2 pad 4: +5V -> Net-(R1-Pad1)
Routing:
- net /SDA: track 403.3 -> 592.0 mm
- net +24V: track 414.8 -> 586.3 mm
- net /SCL: track 475.2 -> 564.7 mm
- net +5V: track 537.3 -> 581.5 mm, vias 0 -> 16
- net /TX: track 0.00 -> 24.3 mm
- net /SEL2: track 63.6 -> 86.3 mm
- net /CSK: track 0.00 -> 20.7 mm
- net /SEL5: track 66.4 -> 84.0 mm
- net Net-(R1-Pad1): track 0.00 -> 15.2 mm
- net /CS: track 0.00 -> 13.5 mm
- net /SEL6: track 35.2 -> 47.8 mm
- net /RX: track 0.00 -> 8.82 mm
- net /SEL1: track 34.1 -> 42.1 mm
- net /RGB_IN: track 4.18 -> 9.87 mm
- net Net-(D17-Pad1): track 25.5 -> 22.2 mm
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Other:
- board text added: "GP1"

Commit message: worked on pcbv1
Parts:
- removed kibuzzard-6233C79C: G***, kibuzzard-6233C79C
- removed kibuzzard-6233C7BC: G***, kibuzzard-6233C7BC
- added kibuzzard-6234ACC3: G***, kibuzzard-6234ACC3, B.Cu at (138.8, 125.6)
- added kibuzzard-6234ACD1: G***, kibuzzard-6234ACD1, B.Cu at (136.2, 125.6)
- added kibuzzard-6234ACE5: G***, kibuzzard-6234ACE5, B.Cu at (133.6, 125.2)
- added kibuzzard-6234ACFA: G***, kibuzzard-6234ACFA, B.Cu at (131.1, 125.1)
- added kibuzzard-6234AD1C: G***, kibuzzard-6234AD1C, B.Cu at (128.6, 125.5)
- added kibuzzard-6234B014: G***, kibuzzard-6234B014, B.Cu at (128.4, 81.6)
- added kibuzzard-6234B02F: G***, kibuzzard-6234B02F, B.Cu at (136.0, 81.4)
- C17: footprint Capacitor_SMD:CP_Elec_8x10 -> Capacitor_SMD:CP_Elec_10x10
- moved J1 4.13 mm to (112.6, 113.7)
- moved J3 3.62 mm to (167.0, 148.6)
- moved J4 3.10 mm to (225.2, 61.7)
- moved J6 1.44 mm to (147.3, 43.5)
- moved C17 1.14 mm to (191.5, 72.3)
- moved J2 1.12 mm to (109.7, 172.1)
- moved J5 1.07 mm to (209.7, 35.1)
Routing:
- net /SEL1: track 42.1 -> 46.8 mm
- net +24V: track 586.3 -> 590.4 mm
- net /SCL: track 564.7 -> 560.8 mm
- net /SEL4: track 77.6 -> 79.9 mm
- net /SEL3: track 40.5 -> 39.2 mm
- net /SEL6: track 47.8 -> 49.0 mm
- net /SDA: track 592.0 -> 591.1 mm
- net /SEL2: track 86.3 -> 87.1 mm
- net /SEL5: track 84.0 -> 83.3 mm
- net +5V: track 581.5 -> 582.1 mm
- net GND: vias 316 -> 339

Commit message: pcb updated
Parts:
- added C19: 1uF, Capacitor_SMD:C_0805_2012Metric, B.Cu at (200.7, 70.3)
- added C20: 100uF, Capacitor_SMD:CP_Elec_10x10.5, B.Cu at (192.8, 72.7)
- added C21: 220uF, Capacitor_SMD:CP_Elec_10x10.5, B.Cu at (190.1, 44.8)
- added C22: 1nF, Capacitor_SMD:C_0805_2012Metric, B.Cu at (181.0, 44.7)
- added C23: 100nF, Capacitor_SMD:C_0805_2012Metric, B.Cu at (181.0, 47.1)
- added C24: 1uF, Capacitor_SMD:C_0805_2012Metric, B.Cu at (181.0, 49.4)
- C17: value 100uF -> 1nF; footprint Capacitor_SMD:CP_Elec_10x10 -> Capacitor_SMD:C_0805_2012Metric
- C18: value 220uF -> 100nF; footprint Capacitor_SMD:CP_Elec_10x10 -> Capacitor_SMD:C_0805_2012Metric
- D17: value 1N5822 -> SS34; footprint Diode_THT:D_DO-201AD_P15.24mm_Horizontal -> Diode_SMD:D_SMC_Handsoldering
- moved C18 28.5 mm to (202.9, 70.3), turned to 90 degrees
- moved C17 13.9 mm to (205.2, 70.3), turned to 90 degrees
- moved D17 10.3 mm to (174.8, 57.8)
- moved C4 8.99 mm to (81.0, 161.3)
- moved C15 8.52 mm to (127.9, 76.2), turned to 90 degrees
- moved C13 3.73 mm to (166.4, 41.8), turned to 90 degrees
- moved C2 3.61 mm to (107.9, 124.3), turned to 90 degrees
- moved C12 1.91 mm to (202.6, 37.7), turned to 180 degrees
- moved C6 1.90 mm to (138.7, 160.8), turned to 0 degrees
- moved C8 1.89 mm to (179.1, 117.8), turned to 90 degrees
Connections:
- C18 pad 1: +5V -> +24V
Routing:
- net +24V: track 590.4 -> 389.6 mm
- net +5V: track 582.1 -> 599.7 mm
- net Net-(D17-Pad1): track 22.2 -> 20.9 mm
- net GND: vias 339 -> 343
- added copper zone on B.Cu, net +24V

Commit message: updated pcb
Parts:
- added R3: 4K7, Resistor_SMD:R_0805_2012Metric, B.Cu at (156.4, 75.4)
- added R4: 4K7, Resistor_SMD:R_0805_2012Metric, B.Cu at (156.4, 73.2)
- C20: footprint Capacitor_SMD:CP_Elec_10x10.5 -> Capacitor_SMD:CP_Elec_6.3x7.7
- C21: footprint Capacitor_SMD:CP_Elec_10x10.5 -> Capacitor_SMD:CP_Elec_8x10.5
- D17: footprint Diode_SMD:D_SMC_Handsoldering -> Diode_SMD:D_SMA_Handsoldering
- moved C20 5.07 mm to (189.2, 69.2)
- moved D17 3.01 mm to (176.7, 60.2)
- moved C21 2.37 mm to (192.2, 45.9)
- moved C17 0.37 mm to (205.2, 69.9)
- moved C18 0.36 mm to (203.0, 69.9)
- moved C19 0.35 mm to (200.8, 69.9)
Connections:
- U1 pad 36: unconnected-(U1-Pad36) -> +3V3
Routing:
- net +24V: track 389.6 -> 25.0 mm
- net +3V3: track 0.00 -> 51.4 mm
- net /SCL: track 560.7 -> 593.4 mm
- net /SDA: track 591.0 -> 623.5 mm
- net Net-(D17-Pad1): track 20.9 -> 18.8 mm
- net GND: vias 343 -> 341
