File: hardware/pcb/pcb_v1/pcb_v1.kicad_sch (KiCad schematic)
At the start: 54 parts, among them J1 Conn_01x10, J2 Conn_01x10, J3 Conn_01x10, J4 Conn_01x10, J5 Conn_01x10, J6 Conn_01x10, J7 Barrel_Jack_Switch, J8 Conn_01x05, U1 Pico, U2 LM2596S-ADJ

Commit message: updated pcb
Parts:
- added R3, R4: 4K7, Resistor_SMD:R_0805_2012Metric, symbol Device:R
- C20: footprint Capacitor_SMD:CP_Elec_10x10.5 -> Capacitor_SMD:CP_Elec_6.3x7.7
- C21: footprint Capacitor_SMD:CP_Elec_10x10.5 -> Capacitor_SMD:CP_Elec_8x10.5
- D17: footprint Diode_SMD:D_SMC_Handsoldering -> Diode_SMD:D_SMA_Handsoldering
Connections:
- net SCL: now also R4.2
- net SDA: now also R3.2
- net +3V3: now reaches U1.36 (3V3)
- net +3V3: now also R3.1, R4.1
- no-connect marks 22 -> 21
Other:
- note added: "EXTERNE I2C PULLUPS"
Changed lines of the file:
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@@
   )
   (no_connect (at 269.24 133.35))
-  (no_connect (at 140.97 39.37))
   (no_connect (at 140.97 41.91))
   (no_connect (at 140.97 54.61))
@@
     (stroke (width 0) (type default) (color 0 0 0 0))
   )
+  (polyline (pts (xy 148.59 114.3) (xy 148.59 91.44))
+    (stroke (width 0) (type default) (color 0 0 0 0))
+  )
   (wire (pts (xy 64.77 27.94) (xy 64.77 48.26))
     (stroke (width 0) (type default) (color 0 0 0 0))
@@
     (stroke (width 0) (type default) (color 0 0 0 0))
   )
+  (wire (pts (xy 139.7 107.95) (xy 139.7 110.49))
+    (stroke (width 0) (type default) (color 0 0 0 0))
+  )
   (wire (pts (xy 68.58 114.3) (xy 68.58 113.03))
     (stroke (width 0) (type default) (color 0 0 0 0))
@@
     (stroke (width 0) (type default) (color 0 0 0 0))
   )
+  (wire (pts (xy 139.7 110.49) (xy 146.05 110.49))
+    (stroke (width 0) (type default) (color 0 0 0 0))
+  )
   (wire (pts (xy 62.23 30.48) (xy 63.5 30.48))
     (stroke (width 0) (type default) (color 0 0 0 0))
@@
     (stroke (width 0) (type default) (color 0 0 0 0))
   )
+  (wire (pts (xy 129.54 107.95) (xy 129.54 110.49))
+    (stroke (width 0) (type default) (color 0 0 0 0))
+  )
   (wire (pts (xy 33.02 64.77) (xy 35.56 64.77))
     (stroke (width 0) (type default) (color 0 0 0 0))
@@
     (stroke (width 0) (type default) (color 0 0 0 0))
   )
+  (wire (pts (xy 129.54 110.49) (xy 135.89 110.49))
+    (stroke (width 0) (type default) (color 0 0 0 0))
+  )
   (wire (pts (xy 259.08 60.96) (xy 261.62 60.96))
     (stroke (width 0) (type default) (color 0 0 0 0))
@@
     (stroke (width 0) (type default) (color 0 0 0 0))
   )
+  (polyline (pts (xy 124.46 114.3) (xy 148.59 114.3))
+    (stroke (width 0) (type default) (color 0 0 0 0))
+  )
   (wire (pts (xy 210.82 60.96) (xy 213.36 60.96))
     (stroke (width 0) (type default) (color 0 0 0 0))
@@
     (stroke (width 0) (type default) (color 0 0 0 0))
   )
+  (polyline (pts (xy 124.46 92.71) (xy 124.46 114.3))
+    (stroke (width 0) (type default) (color 0 0 0 0))
+  )
   (wire (pts (xy 248.92 29.21) (xy 248.92 30.48))
     (stroke (width 0) (type default) (color 0 0 0 0))
@@
     (stroke (width 0) (type default) (color 0 0 0 0))
   )
+  (polyline (pts (xy 124.46 91.44) (xy 124.46 92.71))
+    (stroke (width 0) (type default) (color 0 0 0 0))
+  )
   (wire (pts (xy 213.36 29.21) (xy 213.36 27.94))
     (stroke (width 0) (type default) (color 0 0 0 0))
@@
     (stroke (width 0) (type default) (color 0 0 0 0))
   )
+  (polyline (pts (xy 148.59 91.44) (xy 124.46 91.44))
+    (stroke (width 0) (type default) (color 0 0 0 0))
+  )
   (wire (pts (xy 144.78 29.21) (xy 144.78 31.75))
     (stroke (width 0) (type default) (color 0 0 0 0))
@@
     (effects (font (size 1.27 1.27)) (justify left bottom))
   )
+  (text "EXTERNE I2C PULLUPS" (at 124.46 91.44 0)
+    (effects (font (size 1.27 1.27)) (justify left bottom))
+  )
   (text "VOEDING" (at 17.78 139.7 0)
     (effects (font (size 1.27 1.27)) (justify left bottom))
@@
     (effects (font (size 1.27 1.27)) (justify left bottom))
   )
+  (label "SDA" (at 132.08 110.49 0)
+    (effects (font (size 1.27 1.27)) (justify left bottom))
+  )
   (label "SEL6" (at 69.85 113.03 0)
     (effects (font (size 1.27 1.27)) (justify left bottom))
@@
     (effects (font (size 1.27 1.27)) (justify left bottom))
   )
+  (label "SCL" (at 142.24 110.49 0)
+    (effects (font (size 1.27 1.27)) (justify left bottom))
+  )
   (label "SEL3" (at 40.64 76.2 0)
     (effects (font (size 1.27 1.27)) (justify left bottom))
@@
       (effects (font (size 1.27 1.27)) (justify left))
     )
-    (property "Footprint" "Capacitor_SMD:CP_Elec_10x10.5" (id 2) (at 106.68 162.56 0)
+    (property "Footprint" "Capacitor_SMD:CP_Elec_8x10.5" (id 2) (at 106.68 162.56 0)
       (effects (font (size 1.27 1.27)) hide)
     )
@@
     (pin "2")
   )
+  (symbol (lib_id "Device:R") (at 139.7 104.14 0) (unit 1)
+    (in_bom yes) (on_board yes) (fields_autoplaced)
+    (property "Reference" "R4" (id 0) (at 142.24 102.8699 0)
+      (effects (font (size 1.27 1.27)) (justify left))
+    )
+    (property "Value" "4K7" (id 1) (at 142.24 105.4099 0)
+      (effects (font (size 1.27 1.27)) (justify left))
+    )
+    (property "Footprint" "Resistor_SMD:R_0805_2012Metric" (id 2) (at 137.922 104.14 90)
+      (effects (font (size 1.27 1.27)) hide)
+    )
+    (property "Datasheet" "~" (id 3) (at 139.7 104.14 0)
+      (effects (font (size 1.27 1.27)) hide)
+    )
+    (pin "1")
+    (pin "2")
+  )
   (symbol (lib_id "power:GND") (at 224.79 93.98 0) (unit 1)
     (in_bom yes) (on_board yes)
@@
     (pin "1")
   )
+  (symbol (lib_id "power:+3V3") (at 139.7 100.33 0) (unit 1)
+    (in_bom yes) (on_board yes) (fields_autoplaced)
+    (property "Reference" "#PWR0187" (id 0) (at 139.7 104.14 0)
+      (effects (font (size 1.27 1.27)) hide)
+    )
+    (property "Value" "+3V3" (id 1) (at 139.7 95.25 0))
+    (property "Footprint" "" (id 2) (at 139.7 100.33 0)
+      (effects (font (size 1.27 1.27)) hide)
+    )
+    (property "Datasheet" "" (id 3) (at 139.7 100.33 0)
+      (effects (font (size 1.27 1.27)) hide)
+    )
+    (pin "1")
+  )
   (symbol (lib_id "power:GND") (at 200.66 30.48 0) (unit 1)
     (in_bom yes) (on_board yes)
@@
     (pin "1")
   )
+  (symbol (lib_id "power:+3V3") (at 140.97 39.37 270) (unit 1)
+    (in_bom yes) (on_board yes) (fields_autoplaced)
+    (property "Reference" "#PWR0189" (id 0) (at 137.16 39.37 0)
+      (effects (font (size 1.27 1.27)) hide)
+    )
+    (property "Value" "+3V3" (id 1) (at 144.78 39.3699 90)
+      (effects (font (size 1.27 1.27)) (justify left))
+    )
+    (property "Footprint" "" (id 2) (at 140.97 39.37 0)
+      (effects (font (size 1.27 1.27)) hide)
+    )
+    (property "Datasheet" "" (id 3) (at 140.97 39.37 0)
+      (effects (font (size 1.27 1.27)) hide)
+    )
+    (pin "1")
+  )
   (symbol (lib_id "power:GND") (at 90.17 167.64 0) (unit 1)
     (in_bom yes) (on_board yes) (fields_autoplaced)
@@
       (effects (font (size 1.27 1.27)) (justify left))
     )
-    (property "Footprint" "Diode_SMD:D_SMC_Handsoldering" (id 2) (at 90.17 162.56 0)
+    (property "Footprint" "Diode_SMD:D_SMA_Handsoldering" (id 2) (at 90.17 162.56 0)
       (effects (font (size 1.27 1.27)) hide)
     )
@@
     (pin "1")
   )
+  (symbol (lib_id "Device:R") (at 129.54 104.14 0) (unit 1)
+    (in_bom yes) (on_board yes) (fields_autoplaced)
+    (property "Reference" "R3" (id 0) (at 132.08 102.8699 0)
+      (effects (font (size 1.27 1.27)) (justify left))
+    )
+    (property "Value" "4K7" (id 1) (at 132.08 105.4099 0)
+      (effects (font (size 1.27 1.27)) (justify left))
+    )
+    (property "Footprint" "Resistor_SMD:R_0805_2012Metric" (id 2) (at 127.762 104.14 90)
+      (effects (font (size 1.27 1.27)) hide)
+    )
+    (property "Datasheet" "~" (id 3) (at 129.54 104.14 0)
+      (effects (font (size 1.27 1.27)) hide)
+    )
+    (pin "1")
+    (pin "2")
+  )
   (symbol (lib_id "power:+24V") (at 34.29 100.33 0) (unit 1)
     (in_bom yes) (on_board yes)
@@
     (pin "5")
   )
+  (symbol (lib_id "power:+3V3") (at 129.54 100.33 0) (unit 1)
+    (in_bom yes) (on_board yes) (fields_autoplaced)
+    (property "Reference" "#PWR0188" (id 0) (at 129.54 104.14 0)
+      (effects (font (size 1.27 1.27)) hide)
+    )
+    (property "Value" "+3V3" (id 1) (at 129.54 95.25 0))
+    (property "Footprint" "" (id 2) (at 129.54 100.33 0)
+      (effects (font (size 1.27 1.27)) hide)
+    )
+    (property "Datasheet" "" (id 3) (at 129.54 100.33 0)
+      (effects (font (size 1.27 1.27)) hide)
+    )
+    (pin "1")
+  )
   (symbol (lib_id "Device:C") (at 44.45 160.02 0) (unit 1)
     (in_bom yes) (on_board yes)
@@
       (effects (font (size 1.27 1.27)) (justify left))
     )
-    (property "Footprint" "Capacitor_SMD:CP_Elec_10x10.5" (id 2) (at 53.34 160.02 0)
+    (property "Footprint" "Capacitor_SMD:CP_Elec_6.3x7.7" (id 2) (at 53.34 160.02 0)
       (effects (font (size 1.27 1.27)) hide)
     )
@@
       (reference "#PWR0186") (unit 1) (value "GND") (footprint "")
     )
+    (path "/527fbb99-c4ee-4416-8e53-072053801025"
+      (reference "#PWR0187") (unit 1) (value "+3V3") (footprint "")
+    )
+    (path "/d2733ef0-45ba-42f8-b732-aa16695fb6ef"
+      (reference "#PWR0188") (unit 1) (value "+3V3") (footprint "")
+    )
+    (path "/77101aac-1b93-4115-9c56-a1cc7654c887"
+      (reference "#PWR0189") (unit 1) (value "+3V3") (footprint "")
+    )
     (path "/c4392e1e-f7ba-4051-b85b-627b974eec29"
       (reference "C1") (unit 1) (value "100nF") (footprint "Capacitor_SMD:C_0805_2012Metric")
@@
     )
     (path "/d73b694f-1ab1-4db6-bb3d-f5bad9679bce"
-      (reference "C20") (unit 1) (value "100uF") (footprint "Capacitor_SMD:CP_Elec_10x10.5")
+      (reference "C20") (unit 1) (value "100uF") (footprint "Capacitor_SMD:CP_Elec_6.3x7.7")
     )
     (path "/1ff6d449-c96b-4fec-ab38-4989fc24a6c5"
-      (reference "C21") (unit 1) (value "220uF") (footprint "Capacitor_SMD:CP_Elec_10x10.5")
+      (reference "C21") (unit 1) (value "220uF") (footprint "Capacitor_SMD:CP_Elec_8x10.5")
     )
     (path "/30502310-37df-4a36-94bd-bd3b16f2afe3"
@@
     )
     (path "/876538c4-9b2c-47e3-ba34-df230a80c897"
-      (reference "D17") (unit 1) (value "SS34") (footprint "Diode_SMD:D_SMC_Handsoldering")
+      (reference "D17") (unit 1) (value "SS34") (footprint "Diode_SMD:D_SMA_Handsoldering")
     )
     (path "/2a3f5b67-1280-4816-b0e5-adea4657ddfb"
@@
       (reference "R2") (unit 1) (value "1k") (footprint "Resistor_SMD:R_0805_2012Metric")
     )
+    (path "/9ece809e-238e-4eae-a7ef-e6776d72e441"
+      (reference "R3") (unit 1) (value "4K7") (footprint "Resistor_SMD:R_0805_2012Metric")
+    )
+    (path "/42dfcfdc-f5fb-40d3-80dc-3b68897fd0c1"
+      (reference "R4") (unit 1) (value "4K7") (footprint "Resistor_SMD:R_0805_2012Metric")
+    )
     (path "/716ecf09-84ce-4b48-8ae4-1189810999e9"
